File: Test PCB/GPSDO-LCD-2/GPSDO-LCD-2.sch (KiCad schematic (older format))
At the start: 95 parts, among them J1 Conn_Coaxial, J2 Conn_Coaxial, J3 Conn_Coaxial, J4 Conn_Coaxial, J5 Conn_02x02_Counter_Clockwise, SW1 SW_Push, SW2 SW_Push, SW3 SW_Push, U1 OPA692, U10 Jack_DC, U2 LM1084-ADJ, U3 Arduino_STM32F103C8T6_2, U4 LMP7731, U5 LM1084-ADJ, U6 LCD 16x2, U7 NEO-6M, U8 OCXO-CTI_OSC5A, U9 STP2145A

Commit message: Update
Update
Parts:
- C1, C10, C11, C12, C13, C14, C16, C17, C2, C20, C22, C23, C24, C26, C27, C28, C29, C3, C30, C31, C34, C35, C38, C39, C4, C5, C6, C7, C8: symbol Device:C_Small -> GPSDO-LCD-2-rescue:C_Small-Device
- C15, C18, C19, C21, C25, C32, C33, C36, C37, C9: symbol Device:CP_Small -> GPSDO-LCD-2-rescue:CP_Small-Device
- D1: symbol pspice:DIODE -> GPSDO-LCD-2-rescue:DIODE-pspice
- J1, J2, J3, J4: symbol Connector:Conn_Coaxial -> GPSDO-LCD-2-rescue:Conn_Coaxial-Connector
- J5: symbol Connector_Generic:Conn_02x02_Counter_Clockwise -> GPSDO-LCD-2-rescue:Conn_02x02_Counter_Clockwise-Connector_Generic
- JP1, JP2: symbol Jumper:SolderJumper_3_Open -> GPSDO-LCD-2-rescue:SolderJumper_3_Open-Jumper
- L1, L2, L3: symbol Device:L_Core_Ferrite -> GPSDO-LCD-2-rescue:L_Core_Ferrite-Device
- R1, R10, R11, R12, R13, R14, R15, R16, R17, R18, R19, R2, R20, R21, R22, R23, R24, R25, R26, R27, R28, R29, R3, R30, R31, R32, R4, R5, R6, R7, R8, R9: symbol Device:R -> GPSDO-LCD-2-rescue:R-Device
- SW1, SW2, SW3: symbol Switch:SW_Push -> GPSDO-LCD-2-rescue:SW_Push-Switch
- U1: symbol Personal:OPA692 -> GPSDO-LCD-2-rescue:OPA692-Personal
- U10: symbol Personal:Jack_DC -> GPSDO-LCD-2-rescue:Jack_DC-Personal
- U2, U5: symbol Regulator_Linear:LM1084-ADJ -> GPSDO-LCD-2-rescue:LM1084-ADJ-Regulator_Linear
- U3: symbol Arduino:Arduino_STM32F103C8T6_2 -> GPSDO-LCD-2-rescue:Arduino_STM32F103C8T6_2-Arduino
- U4: symbol Personal:LMP7731 -> GPSDO-LCD-2-rescue:LMP7731-Personal
- U7: symbol Personal:NEO-6M -> GPSDO-LCD-2-rescue:NEO-6M-Personal
- U8: symbol Personal:OCXO-CTI_OSC5A -> GPSDO-LCD-2-rescue:OCXO-CTI_OSC5A-Personal
- U9: symbol Personal:STP2145A -> GPSDO-LCD-2-rescue:STP2145A-Personal
